File: Schematic_&_Board/GaN-amplifier.sch (EAGLE design)
At the start: 108 parts, among them IC1 LT3080, J1 JOHNSON_SMA_EDGE_LAUNCH_142-0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, J2 JOHNSON_SMA_EDGE_LAUNCH_142-0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, Q1 MMBT3906LT1SMD, T1 IPB080N03L G, T2 IPB080N03L G, T3 IPB080N03L G, T4 IPB080N03L G, T5 BSP89, U1 TPS7A30XX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

Commit message: Updates per test board
Adding pulldown on Vdd and On/Off to prevent errors during power
sequencing. Also increasing capacitance of AC coupling capacitors for
better low frequency performance. A couple cosmetic changes to make
component labels visible.

DSB
Parts:
- added R40, R41, R42: 10k, jqi_passives:R_SMDR0603
- C15: value 220n -> 1u; PARTNO CL10B224KP8NNNC -> CL10B105KA8NNNC
- C16: value 150n -> 680n; PARTNO CL10B154KP8NNNC -> CL10B684KO8NFNC
- C23, C24, C6, C7: value 2.2n -> 22n; PARTNO CL10B222KB8NNNC -> CL10B223KB8NNNC
Connections:
- net GND: now also R40.1, R41.1, R42.1
- net N$4: now also R42.2
- net VDD: now also R40.2, R41.2
Changed lines of the file:
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@@
 <attribute name="PARTNO" value="UMK325C7106MM-T"/>
 </part>
-<part name="C6" library="jqi_passives" deviceset="C_MLCC_SMD" device="CMLCC_0603" value="2.2n">
-<attribute name="PARTNO" value="CL10B222KB8NNNC"/>
-</part>
-<part name="C7" library="jqi_passives" deviceset="C_MLCC_SMD" device="CMLCC_0603" value="2.2n">
-<attribute name="PARTNO" value="CL10B222KB8NNNC"/>
+<part name="C6" library="jqi_passives" deviceset="C_MLCC_SMD" device="CMLCC_0603" value="22n">
+<attribute name="PARTNO" value="CL10B223KB8NNNC"/>
+</part>
+<part name="C7" library="jqi_passives" deviceset="C_MLCC_SMD" device="CMLCC_0603" value="22n">
+<attribute name="PARTNO" value="CL10B223KB8NNNC"/>
 </part>
 <part name="GND4" library="supply1" deviceset="GND" device=""/>
@@
 </part>
 <part name="P+4" library="supply1" deviceset="+5V" device=""/>
-<part name="C15" library="jqi_passives" deviceset="C_MLCC_SMD" device="CMLCC_0603" value="220n">
-<attribute name="PARTNO" value="CL10B224KP8NNNC"/>
-</part>
-<part name="C16" library="jqi_passives" deviceset="C_MLCC_SMD" device="CMLCC_0603" value="150n">
-<attribute name="PARTNO" value="CL10B154KP8NNNC"/>
+<part name="C15" library="jqi_passives" deviceset="C_MLCC_SMD" device="CMLCC_0603" value="1u">
+<attribute name="PARTNO" value="CL10B105KA8NNNC"/>
+</part>
+<part name="C16" library="jqi_passives" deviceset="C_MLCC_SMD" device="CMLCC_0603" value="680n">
+<attribute name="PARTNO" value="CL10B684KO8NFNC"/>
 </part>
 <part name="R4" library="jqi_passives" deviceset="R_SMD" device="R0603" value="49.9k">
@@
 <attribute name="PARTNO" value="LVK12R050DER"/>
 </part>
-<part name="C23" library="jqi_passives" deviceset="C_MLCC_SMD" device="CMLCC_0603" value="2.2n">
-<attribute name="PARTNO" value="CL10B222KB8NNNC"/>
-</part>
-<part name="C24" library="jqi_passives" deviceset="C_MLCC_SMD" device="CMLCC_0603" value="2.2n">
-<attribute name="PARTNO" value="CL10B222KB8NNNC"/>
+<part name="C23" library="jqi_passives" deviceset="C_MLCC_SMD" device="CMLCC_0603" value="22n">
+<attribute name="PARTNO" value="CL10B223KB8NNNC"/>
+</part>
+<part name="C24" library="jqi_passives" deviceset="C_MLCC_SMD" device="CMLCC_0603" value="22n">
+<attribute name="PARTNO" value="CL10B223KB8NNNC"/>
 </part>
 <part name="GND3" library="supply1" deviceset="GND" device=""/>
@@
 <attribute name="PARTNO" value="CL10B104KB8SFNC"/>
 </part>
+<part name="R40" library="jqi_passives" deviceset="R_SMD" device="R0603" value="10k">
+<attribute name="PARTNO" value="ERJ-3EKF1002V"/>
+</part>
+<part name="R41" library="jqi_passives" deviceset="R_SMD" device="R0603" value="10k">
+<attribute name="PARTNO" value="ERJ-3EKF1002V"/>
+</part>
+<part name="R42" library="jqi_passives" deviceset="R_SMD" device="R0603" value="10k">
+<attribute name="PARTNO" value="ERJ-3EKF1002V"/>
+</part>
+<part name="GND23" library="supply1" deviceset="GND" device=""/>
 </parts>
 <sheets>
@@
 <attribute name="PARTNO" x="31.75" y="78.74" size="1.778" layer="96" display="off"/>
 </instance>
+<instance part="R40" gate="G$1" x="246.38" y="168.91" rot="R90">
+<attribute name="PARTNO" x="246.38" y="168.91" size="1.778" layer="96" display="off"/>
+</instance>
+<instance part="R41" gate="G$1" x="251.46" y="168.91" rot="R90">
+<attribute name="PARTNO" x="251.46" y="168.91" size="1.778" layer="96" display="off"/>
+</instance>
+<instance part="R42" gate="G$1" x="124.46" y="180.34" rot="R180">
+<attribute name="PARTNO" x="124.46" y="180.34" size="1.778" layer="96" rot="R90" display="off"/>
+</instance>
+<instance part="GND23" gate="1" x="251.46" y="156.21"/>
 </instances>
 <busses>
@@
 <wire x1="157.48" y1="158.75" x2="166.37" y2="158.75" width="0.1524" layer="91"/>
 <wire x1="166.37" y1="158.75" x2="166.37" y2="162.56" width="0.1524" layer="91"/>
+<pinref part="R42" gate="G$1" pin="1"/>
+<wire x1="129.54" y1="180.34" x2="168.91" y2="180.34" width="0.1524" layer="91"/>
+<wire x1="168.91" y1="180.34" x2="168.91" y2="158.75" width="0.1524" layer="91"/>
+<wire x1="168.91" y1="158.75" x2="166.37" y2="158.75" width="0.1524" layer="91"/>
+<junction x="166.37" y="158.75"/>
 </segment>
 <segment>
@@
 <pinref part="C19" gate="G$1" pin="P$1"/>
 <pinref part="C20" gate="G$1" pin="P$2"/>
+</segment>
+<segment>
+<pinref part="R40" gate="G$1" pin="1"/>
+<wire x1="246.38" y1="163.83" x2="246.38" y2="161.29" width="0.1524" layer="91"/>
+<wire x1="246.38" y1="161.29" x2="251.46" y2="161.29" width="0.1524" layer="91"/>
+<pinref part="R41" gate="G$1" pin="1"/>
+<wire x1="251.46" y1="161.29" x2="251.46" y2="163.83" width="0.1524" layer="91"/>
+<pinref part="GND23" gate="1" pin="GND"/>
+<wire x1="251.46" y1="161.29" x2="251.46" y2="158.75" width="0.1524" layer="91"/>
+<junction x="251.46" y="161.29"/>
 </segment>
 </net>
@@
 <wire x1="127" y1="189.23" x2="113.03" y2="189.23" width="0.1524" layer="91"/>
 <wire x1="113.03" y1="189.23" x2="113.03" y2="180.34" width="0.1524" layer="91"/>
+<pinref part="R42" gate="G$1" pin="2"/>
+<wire x1="113.03" y1="180.34" x2="119.38" y2="180.34" width="0.1524" layer="91"/>
+<junction x="113.03" y="180.34"/>
 </segment>
 </net>
@@
 <wire x1="222.25" y1="176.53" x2="224.79" y2="176.53" width="0.1524" layer="91"/>
 <wire x1="224.79" y1="176.53" x2="224.79" y2="172.72" width="0.1524" layer="91"/>
-<wire x1="224.79" y1="176.53" x2="232.41" y2="176.53" width="0.1524" layer="91"/>
 <junction x="224.79" y="176.53"/>
 <label x="227.33" y="176.53" size="1.778" layer="95"/>
-</segment>
-</net>
+<pinref part="R40" gate="G$1" pin="2"/>
+<wire x1="224.79" y1="176.53" x2="246.38" y2="176.53" width="0.1524" layer="91"/>
+<wire x1="246.38" y1="176.53" x2="246.38" y2="173.99" width="0.1524" layer="91"/>
+<pinref part="R41" gate="G$1" pin="2"/>
+<wire x1="246.38" y1="176.53" x2="251.46" y2="176.53" width="0.1524" layer="91"/>
+<wire x1="251.46" y1="176.53" x2="251.46" y2="173.99" width="0.1524" layer="91"/>
+<junction x="246.38" y="176.53"/>
+</segment>
+</net>
